File: HB-RF-MOD.kicad_pcb (KiCad board)
At the start: 2 copper layers, 36.2 x 65 mm, 25 parts, among them J1 RPi Header, J2 RGB, Q1 BC847, SW1 Button, U1 TRX2-TIF, U2 RX8130-CE, U3 3V3LDO

Commit message: update
Parts:
- moved R2 4.98 mm to (177.7, 94.5), turned to 270 degrees
- moved J2 4.65 mm to (187.4, 113.4)
- moved C6 1.69 mm to (184.2, 96.0), turned to 90 degrees
- moved C4 0.92 mm to (174.1, 104.7)
- moved U3 0.65 mm to (185.3, 61.2)
- moved C5 0.45 mm to (180.2, 60.2)
- moved C7 0.43 mm to (173.7, 61.2)
- moved C1 0.25 mm to (185.1, 73.3)
- moved R9 0.20 mm to (162.4, 93.1)
- moved C2 0.20 mm to (182.6, 73.3)
Routing:
- net GND: track 174.1 -> 28.2 mm, vias 6 -> 30
- net RESET: track 27.9 -> 21.5 mm
- net +5V: track 71.6 -> 65.9 mm
- net BUTTON: track 20.7 -> 22.0 mm
- net Net-(Q1-Pad1): track 19.3 -> 18.2 mm
- net Net-(J1-Pad40): track 8.13 -> 8.88 mm
- added copper zone on F.Cu, net +5V
Other:
- board size 36.2 x 65 mm -> 35.6 x 64.2 mm
- board text added: "+5V"
- board text added: "B"
- board text added: "G"
- board text added: "GND"
- board text added: "R"

Commit message: update
Routing:
- net GND: track 28.2 -> 21.6 mm, vias 30 -> 34
Changed lines of the file:
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@@
     (thickness 1.6)
     (drawings 13)
-    (tracks 241)
+    (tracks 238)
     (zones 0)
     (modules 25)
@@
     (mod_text_size 1 1)
     (mod_text_width 0.15)
-    (pad_size 1.524 1.524)
-    (pad_drill 0.762)
+    (pad_size 1 1.5)
+    (pad_drill 0)
     (pad_to_mask_clearance 0)
     (aux_axis_origin 0 0)
@@
     (descr SOT-89-3)
     (tags SOT-89-3)
+    (zone_connect 2)
     (attr smd)
     (fp_text reference U3 (at 4.1 0 90) (layer F.SilkS)
@@
     )
     (pad 2 smd trapezoid (at -0.0762 0 90) (size 1.5 1) (rect_delta 0 0.7 ) (layers F.Cu F.Paste F.Mask)
-      (net 48 +5V))
+      (net 48 +5V) (zone_connect 2))
     (pad 2 smd rect (at 1.3335 0 270) (size 2.2 1.84) (layers F.Cu F.Paste F.Mask)
-      (net 48 +5V))
+      (net 48 +5V) (zone_connect 2))
     (pad 3 smd rect (at -1.48 1.5 270) (size 1 1.5) (layers F.Cu F.Paste F.Mask)
-      (net 17 +3V3))
+      (net 17 +3V3) (zone_connect 2))
     (pad 2 smd rect (at -1.3335 0 270) (size 1 1.8) (layers F.Cu F.Paste F.Mask)
-      (net 48 +5V))
+      (net 48 +5V) (zone_connect 2))
     (pad 1 smd rect (at -1.48 -1.5 270) (size 1 1.5) (layers F.Cu F.Paste F.Mask)
-      (net 16 GND))
+      (net 16 GND) (zone_connect 1))
     (pad 2 smd trapezoid (at 2.667 0 270) (size 1.6 0.85) (rect_delta 0 0.6 ) (layers F.Cu F.Paste F.Mask)
-      (net 48 +5V))
+      (net 48 +5V) (zone_connect 2))
     (model ${KISYS3DMOD}/Package_TO_SOT_SMD.3dshapes/SOT-89-3.wrl
       (at (xyz 0 0 0))
@@
   (segment (start 186.69 89.2353) (end 186.5003 89.425) (width 0.25) (layer F.Cu) (net 16))
   (segment (start 185.65 89.425) (end 186.5003 89.425) (width 0.25) (layer F.Cu) (net 16))
-  (segment (start 194.29 80.44) (end 194.29 79.2647) (width 0.25) (layer F.Cu) (net 16))
-  (segment (start 191.75 75.36) (end 191.75 76.5353) (width 0.25) (layer F.Cu) (net 16))
-  (segment (start 191.75 76.5353) (end 192.1174 76.5353) (width 0.25) (layer F.Cu) (net 16))
-  (segment (start 192.1174 76.5353) (end 193.1147 77.5326) (width 0.25) (layer F.Cu) (net 16))
-  (segment (start 193.1147 77.5326) (end 193.1147 78.4568) (width 0.25) (layer F.Cu) (net 16))
-  (segment (start 193.1147 78.4568) (end 193.9226 79.2647) (width 0.25) (layer F.Cu) (net 16))
-  (segment (start 193.9226 79.2647) (end 194.29 79.2647) (width 0.25) (layer F.Cu) (net 16))
   (segment (start 165.55 94.2) (end 165.55 95.0753) (width 0.25) (layer F.Cu) (net 16))
   (segment (start 184.4099 89.0352) (end 184.7997 89.425) (width 0.25) (layer F.Cu) (net 16))
@@
   (via (at 174.6 91.175) (size 0.8) (drill 0.4) (layers F.Cu B.Cu) (net 16))
   (via (at 174.55 94.25) (size 0.8) (drill 0.4) (layers F.Cu B.Cu) (net 16))
+  (via (at 190.9 58.65) (size 0.8) (drill 0.4) (layers F.Cu B.Cu) (net 16))
+  (via (at 194.825 62.925) (size 0.8) (drill 0.4) (layers F.Cu B.Cu) (net 16))
+  (via (at 194.925 115.825) (size 0.8) (drill 0.4) (layers F.Cu B.Cu) (net 16))
+  (via (at 190.775 119.9) (size 0.8) (drill 0.4) (layers F.Cu B.Cu) (net 16))
   (segment (start 169.1299 88.6799) (end 169.1299 90.3013) (width 0.25) (layer F.Cu) (net 17))
   (segment (start 169.1299 90.3013) (end 168.3065 91.1247) (width 0.25) (layer F.Cu) (net 17))

Commit message: update
Routing:
- net GND: track 21.6 -> 16.0 mm
Changed lines of the file:
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@@
     (thickness 1.6)
     (drawings 13)
-    (tracks 238)
+    (tracks 231)
     (zones 0)
     (modules 25)
@@
     (tags "SPST Button Switch")
     (attr smd)
-    (fp_text reference SW1 (at 0 -2.6) (layer F.SilkS)
+    (fp_text reference SW1 (at 3.645 0.01 90) (layer F.SilkS)
       (effects (font (size 1 1) (thickness 0.15)))
     )
@@
     (tags "resistor handsolder")
     (attr smd)
-    (fp_text reference R5 (at 0 -1.65 90) (layer F.SilkS)
+    (fp_text reference R5 (at 0.2 1.8 90) (layer F.SilkS)
       (effects (font (size 1 1) (thickness 0.15)))
     )
@@
     (tags "resistor handsolder")
     (attr smd)
-    (fp_text reference R4 (at 0 -1.65 90) (layer F.SilkS)
+    (fp_text reference R4 (at -0.05 1.775 90) (layer F.SilkS)
       (effects (font (size 1 1) (thickness 0.15)))
     )
@@
     (tags SOT-23)
     (attr smd)
-    (fp_text reference Q1 (at 0 -2.5 90) (layer F.SilkS)
+    (fp_text reference Q1 (at -2.475 0.125 90) (layer F.SilkS)
       (effects (font (size 1 1) (thickness 0.15)))
     )
@@
   (gr_line (start 160.894949 120.400013) (end 160.9 58.2) (layer Edge.Cuts) (width 0.1))
   (gr_line (start 195.5 121.4) (end 161.9 121.4) (layer Edge.Cuts) (width 0.1))
-  (segment (start 186.69 89.2353) (end 186.5003 89.425) (width 0.25) (layer F.Cu) (net 16))
-  (segment (start 185.65 89.425) (end 186.5003 89.425) (width 0.25) (layer F.Cu) (net 16))
   (segment (start 165.55 94.2) (end 165.55 95.0753) (width 0.25) (layer F.Cu) (net 16))
-  (segment (start 184.4099 89.0352) (end 184.7997 89.425) (width 0.25) (layer F.Cu) (net 16))
-  (segment (start 184.4099 89.0352) (end 182.7401 89.0352) (width 0.25) (layer F.Cu) (net 16))
-  (segment (start 182.7401 89.0352) (end 182.3503 89.425) (width 0.25) (layer F.Cu) (net 16))
-  (segment (start 181.5 89.425) (end 182.3503 89.425) (width 0.25) (layer F.Cu) (net 16))
   (segment (start 180.475 59.05) (end 180.15 58.725) (width 0.25) (layer F.Cu) (net 16))
-  (segment (start 185.65 89.425) (end 184.7997 89.425) (width 0.25) (layer F.Cu) (net 16))
   (segment (start 185.3 77.2373) (end 185.3 77.6) (width 0.25) (layer F.Cu) (net 16))
   (segment (start 185.3 77.2373) (end 185.3 76.8747) (width 0.25) (layer F.Cu) (net 16))

Commit message: update
Parts:
- added D1: LED_RGBA, LED_THT:LED_D5.0mm-4_RGB_Wide_Pins, F.Cu at (26.9, 69.5)
- added J3: GND, TestPoint:TestPoint_Pad_D1.5mm, F.Cu at (50.1, 30.1)
- added J4: RESET, TestPoint:TestPoint_Pad_D1.5mm, F.Cu at (50.1, 37.6)
- added J5: J_TCKC, TestPoint:TestPoint_Pad_D1.5mm, F.Cu at (50.1, 35.1)
- added J6: J_TMSC, TestPoint:TestPoint_Pad_D1.5mm, F.Cu at (50.1, 32.6)
- added Q2: BC847, Package_TO_SOT_SMD:SOT-23, F.Cu at (38.3, 67.8)
- added Q3: BC847, Package_TO_SOT_SMD:SOT-23, F.Cu at (38.3, 72.3)
- added Q4: BC847, Package_TO_SOT_SMD:SOT-23, F.Cu at (38.2, 77.0)
- added R10: 10k, Resistor_SMD:R_0805_2012Metric_Pad1.15x1.40mm_HandSolder, F.Cu at (47.9, 67.7)
- added R11: 10k, Resistor_SMD:R_0805_2012Metric_Pad1.15x1.40mm_HandSolder, F.Cu at (43.1, 67.6)
- added R12: 10k, Resistor_SMD:R_0805_2012Metric_Pad1.15x1.40mm_HandSolder, F.Cu at (48.0, 72.3)
- added R13: 10k, Resistor_SMD:R_0805_2012Metric_Pad1.15x1.40mm_HandSolder, F.Cu at (43.2, 72.1)
- added R14: 10k, Resistor_SMD:R_0805_2012Metric_Pad1.15x1.40mm_HandSolder, F.Cu at (48.0, 76.6)
- added R15: 10k, Resistor_SMD:R_0805_2012Metric_Pad1.15x1.40mm_HandSolder, F.Cu at (43.1, 76.7)
- added R16: 180, Resistor_SMD:R_0805_2012Metric_Pad1.15x1.40mm_HandSolder, F.Cu at (32.5, 67.8)
- added R17: 100, Resistor_SMD:R_0805_2012Metric_Pad1.15x1.40mm_HandSolder, F.Cu at (32.7, 72.4)
- added R18: 100, Resistor_SMD:R_0805_2012Metric_Pad1.15x1.40mm_HandSolder, F.Cu at (32.8, 77.0)
- C4: footprint Capacitor_THT:CP_Radial_D22.0mm_P10.00mm_SnapIn -> additional:CP_Radial_D20.0mm_P5.00mm; moved to B.Cu
- C7: moved to B.Cu
- J2: value RGB -> 3V3; footprint Connector_PinHeader_2.00mm:PinHeader_1x05_P2.00mm_Vertical -> TestPoint:TestPoint_Pad_D1.5mm
- moved J2 161.9 mm to (50.1, 27.6), turned to 0 degrees
- moved U3 158.7 mm to (32.0, 20.2), turned to 90 degrees
- moved C5 156.9 mm to (28.3, 20.8), turned to 270 degrees
- moved C6 145.9 mm to (44.4, 54.2), turned to 270 degrees
- moved C1 145.5 mm to (46.0, 30.4)
- moved C2 145.3 mm to (43.8, 30.4)
- moved R8 145.1 mm to (48.6, 53.2), turned to 180 degrees
- moved R1 144.6 mm to (45.0, 44.8)
- moved Q1 144.4 mm to (44.9, 41.0)
- moved R2 144.3 mm to (39.5, 53.1)
- moved H1 144.3 mm to (54.8, 76.5)
- moved H2 144.3 mm to (54.8, 19.3)
- moved J1 144.3 mm to (53.5, 23.8)
- moved R3 144.3 mm to (39.4, 49.1)
- moved R5 144.3 mm to (29.9, 47.3)
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Connections:
- J1 pad 36: Net-(J1-Pad36) -> RGB-RED
- J1 pad 38: Net-(J1-Pad38) -> RGB-GREEN
- J1 pad 40: Net-(J1-Pad40) -> RGB-BLUE
- J2 pad 1: GND -> +3V3
Routing:
- net GND: track 16.0 -> 82.6 mm, vias 34 -> 30
- net +5V: track 65.9 -> 99.0 mm, vias 0 -> 2
- net Net-(J4-Pad1): track 10.9 -> 43.1 mm
- net Net-(J6-Pad1): track 0.00 -> 10.7 mm
- net Net-(J5-Pad1): track 0.00 -> 10.2 mm
- net RGB-BLUE: track 0.00 -> 9.15 mm
- net Net-(J1-Pad40): track 8.88 -> 0.00 mm
- net Net-(J1-Pad38): track 8.66 -> 0.00 mm
- net Net-(J1-Pad36): track 8.43 -> 0.00 mm
- net RGB-GREEN: track 0.00 -> 8.42 mm
- net Net-(Q4-Pad1): track 0.00 -> 8.32 mm
- net Net-(Q3-Pad1): track 0.00 -> 8.08 mm
- net RGB-RED: track 0.00 -> 8.04 mm
- net Net-(Q2-Pad1): track 0.00 -> 7.98 mm
- net +3V3: track 117.0 -> 109.1 mm, vias 0 -> 3
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Other:
- net class 5V added: clearance 0.2, trace_width 0.4, via_dia 0.8, via_drill 0.4
- board text added: "1"
- board text added: "1 - RESET 2 - TCKC 3 - TMSC 4 - GND 5 - 3.3V"
- board text added: "2"
- board text added: "3"
- board text added: "4"
- board text added: "5"
- board text removed: "+5V"
- board text removed: "B"
- board text removed: "G"
- board text removed: "GND"
- board text removed: "R"

Commit message: update
Parts:
- moved C5 0.50 mm to (27.8, 20.8)
Routing:
- net +5V: track 99.0 -> 101.9 mm
- net GND: track 82.6 -> 82.0 mm
Changed lines of the file:
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@@
     (thickness 1.6)
     (drawings 23)
-    (tracks 354)
+    (tracks 356)
     (zones 0)
     (modules 42)
@@
   )
   (setup
-    (last_trace_width 0.25)
+    (last_trace_width 0.4)
     (user_trace_width 0.4)
     (trace_clearance 0.2)
@@
   )
   (module Capacitor_SMD:C_0805_2012Metric_Pad1.15x1.40mm_HandSolder (layer F.Cu)
-    (at 28.3 20.8 270)
+    (at 27.8 20.8 270)
     (descr "Capacitor SMD 0805 (2012 Metric), square (rectangular) end terminal, IPC_7351 nominal with elongated pad for handsoldering. (Body size source: https://docs.google.com/spreadsheets/d/1BsfQQcO9C6DZCsRaXUlFlo91Tg2WpOkGARC1WS5S8t0/edit?usp=sharing), generated with kicad-footprint-generator")
     (tags "capacitor handsolder")
@@
   (segment (start 56.07 38.4323) (end 56.07 37.8447) (width 0.25) (layer F.Cu) (net 14))
   (segment (start 43.0723 71.0073) (end 43.16 71.095) (width 0.25) (layer F.Cu) (net 14))
-  (segment (start 28.6926 22.2176) (end 28.3 21.825) (width 0.25) (layer F.Cu) (net 14))
   (segment (start 30.5 21.68) (end 30.5 22.2176) (width 0.25) (layer F.Cu) (net 14))
   (segment (start 53.53 33.94) (end 53.53 35.1153) (width 0.25) (layer F.Cu) (net 14))
@@
   (segment (start 50.8693 25.0697) (end 54.0875 25.0697) (width 0.4) (layer F.Cu) (net 42))
   (segment (start 54.0875 25.0697) (end 54.8197 25.8019) (width 0.4) (layer F.Cu) (net 42))
-  (segment (start 29.4658 18.3962) (end 28.3 19.562) (width 0.4) (layer F.Cu) (net 42))
   (segment (start 28.3 19.562) (end 28.3 19.775) (width 0.4) (layer F.Cu) (net 42))
   (segment (start 50.2178 32.9237) (end 51.0664 33.7723) (width 0.4) (layer B.Cu) (net 42))
@@
   (via (at 50.9984 43.4947) (size 0.8) (layers F.Cu B.Cu) (net 42))
   (via (at 51.0664 33.7723) (size 0.8) (layers F.Cu B.Cu) (net 42))
+  (segment (start 28.5 19.775) (end 28.525 19.8) (width 0.4) (layer F.Cu) (net 42))
+  (segment (start 27.8 19.775) (end 28.5 19.775) (width 0.4) (layer F.Cu) (net 42))
+  (segment (start 28.525 19.8) (end 31.2 19.8) (width 0.4) (layer F.Cu) (net 42))
+  (segment (start 31.2 19.8) (end 32 19) (width 0.4) (layer F.Cu) (net 42))
   (segment (start 53.53 66.96) (end 52.26 66.96) (width 0.25) (layer F.Cu) (net 43))
   (segment (start 52.26 62.886998) (end 46.173002 56.8) (width 0.25) (layer F.Cu) (net 43))

Commit message: update
Routing:
- net GND: track 82.0 -> 40.6 mm
Changed lines of the file:
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@@
     (thickness 1.6)
     (drawings 23)
-    (tracks 356)
+    (tracks 319)
     (zones 0)
     (modules 42)
@@
   (segment (start 49.6253 48.225) (end 50.8074 47.0429) (width 0.25) (layer F.Cu) (net 14))
   (segment (start 50.8074 47.0429) (end 50.8074 45.5514) (width 0.25) (layer F.Cu) (net 14))
-  (segment (start 54.8947 44.6568) (end 54.1181 45.4334) (width 0.25) (layer F.Cu) (net 14))
-  (segment (start 54.1181 45.4334) (end 50.9254 45.4334) (width 0.25) (layer F.Cu) (net 14))
   (segment (start 50.9254 45.4334) (end 50.8074 45.5514) (width 0.25) (layer F.Cu) (net 14))
   (segment (start 43.4512 75.3388) (end 43.135 75.655) (width 0.25) (layer F.Cu) (net 14))
@@
   (segment (start 52.2958 31.9026) (end 52.2958 30.7588) (width 0.25) (layer F.Cu) (net 14))
   (segment (start 56.07 28.86) (end 54.8947 28.86) (width 0.25) (layer F.Cu) (net 14))
-  (segment (start 54.8947 44.6568) (end 55.7026 45.4647) (width 0.25) (layer F.Cu) (net 14))
-  (segment (start 55.7026 45.4647) (end 56.07 45.4647) (width 0.25) (layer F.Cu) (net 14))
-  (segment (start 56.07 40.1953) (end 55.7026 40.1953) (width 0.25) (layer F.Cu) (net 14))
-  (segment (start 55.7026 40.1953) (end 54.8947 41.0032) (width 0.25) (layer F.Cu) (net 14))
-  (segment (start 54.8947 41.0032) (end 54.8947 44.6568) (width 0.25) (layer F.Cu) (net 14))
   (segment (start 48.775 48.225) (end 49.6253 48.225) (width 0.25) (layer F.Cu) (net 14))
-  (segment (start 56.07 39.02) (end 56.07 40.1953) (width 0.25) (layer F.Cu) (net 14))
   (segment (start 56.07 39.02) (end 56.07 38.4323) (width 0.25) (layer F.Cu) (net 14))
-  (segment (start 56.07 46.64) (end 56.07 45.4647) (width 0.25) (layer F.Cu) (net 14))
   (segment (start 53.53 33.94) (end 53.53 32.7647) (width 0.25) (layer F.Cu) (net 14))
   (segment (start 27.33 52.78) (end 27.33 55.255) (width 0.25) (layer F.Cu) (net 14))
   (segment (start 27.33 55.255) (end 29.9 57.825) (width 0.25) (layer F.Cu) (net 14))
-  (segment (start 56.07 59.34) (end 56.07 58.1647) (width 0.25) (layer B.Cu) (net 14))
-  (segment (start 53.53 54.26) (end 53.53 55.4353) (width 0.25) (layer B.Cu) (net 14))
-  (segment (start 53.53 55.4353) (end 53.8974 55.4353) (width 0.25) (layer B.Cu) (net 14))
-  (segment (start 53.8974 55.4353) (end 54.8947 56.4326) (width 0.25) (layer B.Cu) (net 14))
-  (segment (start 54.8947 56.4326) (end 54.8947 57.3568) (width 0.25) (layer B.Cu) (net 14))
-  (segment (start 54.8947 57.3568) (end 55.7026 58.1647) (width 0.25) (layer B.Cu) (net 14))
-  (segment (start 55.7026 58.1647) (end 56.07 58.1647) (width 0.25) (layer B.Cu) (net 14))
-  (segment (start 56.07 64.42) (end 56.07 63.2447) (width 0.25) (layer B.Cu) (net 14))
-  (segment (start 56.07 59.34) (end 56.07 60.5153) (width 0.25) (layer B.Cu) (net 14))
-  (segment (start 56.07 60.5153) (end 55.7027 60.5153) (width 0.25) (layer B.Cu) (net 14))
-  (segment (start 55.7027 60.5153) (end 54.8947 61.3233) (width 0.25) (layer B.Cu) (net 14))
-  (segment (start 54.8947 61.3233) (end 54.8947 62.4368) (width 0.25) (layer B.Cu) (net 14))
-  (segment (start 54.8947 62.4368) (end 55.7026 63.2447) (width 0.25) (layer B.Cu) (net 14))
-  (segment (start 55.7026 63.2447) (end 56.07 63.2447) (width 0.25) (layer B.Cu) (net 14))
-  (segment (start 56.07 38.4323) (end 56.07 37.8447) (width 0.25) (layer F.Cu) (net 14))
   (segment (start 43.0723 71.0073) (end 43.16 71.095) (width 0.25) (layer F.Cu) (net 14))
   (segment (start 30.5 21.68) (end 30.5 22.2176) (width 0.25) (layer F.Cu) (net 14))
-  (segment (start 53.53 33.94) (end 53.53 35.1153) (width 0.25) (layer F.Cu) (net 14))
-  (segment (start 53.53 35.1153) (end 53.8974 35.1153) (width 0.25) (layer F.Cu) (net 14))
-  (segment (start 53.8974 35.1153) (end 54.7053 35.9232) (width 0.25) (layer F.Cu) (net 14))
-  (segment (start 54.7053 35.9232) (end 54.7053 36.8474) (width 0.25) (layer F.Cu) (net 14))
-  (segment (start 54.7053 36.8474) (end 55.7026 37.8447) (width 0.25) (layer F.Cu) (net 14))
-  (segment (start 55.7026 37.8447) (end 56.07 37.8447) (width 0.25) (layer F.Cu) (net 14))
   (segment (start 44.625 48.225) (end 43.7747 48.225) (width 0.25) (layer F.Cu) (net 14))
   (segment (start 40.785 32.955) (end 40.785 32.125) (width 0.25) (layer F.Cu) (net 14))
   (segment (start 40.785 33.395) (end 40.785 32.955) (width 0.25) (layer F.Cu) (net 14))
   (segment (start 44.625 48.225) (end 45.4753 48.225) (width 0.25) (layer F.Cu) (net 14))
-  (segment (start 56.07 64.42) (end 56.07 65.5953) (width 0.25) (layer B.Cu) (net 14))
-  (segment (start 53.53 72.04) (end 53.53 70.8647) (width 0.25) (layer B.Cu) (net 14))
-  (segment (start 53.53 70.8647) (end 53.8974 70.8647) (width 0.25) (layer B.Cu) (net 14))
-  (segment (start 53.8974 70.8647) (end 54.8947 69.8674) (width 0.25) (layer B.Cu) (net 14))
-  (segment (start 54.8947 69.8674) (end 54.8947 66.4032) (width 0.25) (layer B.Cu) (net 14))
-  (segment (start 54.8947 66.4032) (end 55.7026 65.5953) (width 0.25) (layer B.Cu) (net 14))
-  (segment (start 55.7026 65.5953) (end 56.07 65.5953) (width 0.25) (layer B.Cu) (net 14))
   (via (at 49.05 62.25) (size 0.8) (drill 0.4) (layers F.Cu B.Cu) (net 14))
   (via (at 34.8 47.2) (size 0.8) (drill 0.4) (layers F.Cu B.Cu) (net 14))
