File: HB-RF-MOD.kicad_pcb (KiCad board)
At the start: 2 copper layers, 35.6 x 64.2 mm, 42 parts, among them J1 RPi Header, J2 3V3, J3 GND, J4 RESET, J5 J_TCKC, J6 J_TMSC, Q1 BC847, Q2 BC847, Q3 BC847, Q4 BC847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

Commit message: update
Parts:
- moved R7 1.23 mm to (25.2, 55.9), turned to 180 degrees
- moved C4 0.81 mm to (38.4, 60.8)
- moved R18 0.19 mm to (32.6, 77.0)
- moved R17 0.07 mm to (32.6, 72.4)
Routing:
- net +3V3: track 109.1 -> 106.6 mm
- net GND: vias 30 -> 31
Changed lines of the file:
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@@
   )
   (setup
-    (last_trace_width 0.4)
+    (last_trace_width 0.25)
     (user_trace_width 0.4)
     (trace_clearance 0.2)
@@
   )
   (module additional:CP_Radial_D20.0mm_P5.00mm (layer B.Cu)
-    (at 38.8 61.5)
+    (at 38.4 60.8)
     (descr "CP, Radial series, Radial, pin pitch=5.00mm, , diameter=14mm, Electrolytic Capacitor")
     (tags "CP Radial series Radial pin pitch 5.00mm  diameter 14mm Electrolytic Capacitor")
@@
   )
   (module Resistor_SMD:R_0805_2012Metric_Pad1.15x1.40mm_HandSolder (layer F.Cu)
-    (at 32.79 77)
+    (at 32.6 77)
     (descr "Resistor SMD 0805 (2012 Metric), square (rectangular) end terminal, IPC_7351 nominal with elongated pad for handsoldering. (Body size source: https://docs.google.com/spreadsheets/d/1BsfQQcO9C6DZCsRaXUlFlo91Tg2WpOkGARC1WS5S8t0/edit?usp=sharing), generated with kicad-footprint-generator")
     (tags "resistor handsolder")
@@
   )
   (module Resistor_SMD:R_0805_2012Metric_Pad1.15x1.40mm_HandSolder (layer F.Cu)
-    (at 32.67 72.41 180)
+    (at 32.6 72.4 180)
     (descr "Resistor SMD 0805 (2012 Metric), square (rectangular) end terminal, IPC_7351 nominal with elongated pad for handsoldering. (Body size source: https://docs.google.com/spreadsheets/d/1BsfQQcO9C6DZCsRaXUlFlo91Tg2WpOkGARC1WS5S8t0/edit?usp=sharing), generated with kicad-footprint-generator")
     (tags "resistor handsolder")
@@
     (tags "resistor handsolder")
     (attr smd)
-    (fp_text reference R9 (at 2.85 -0.125 90) (layer F.SilkS)
+    (fp_text reference R9 (at -2.705 0.38 90) (layer F.SilkS)
       (effects (font (size 1 1) (thickness 0.15)))
     )
@@
   )
   (module Resistor_SMD:R_0805_2012Metric_Pad1.15x1.40mm_HandSolder (layer F.Cu)
-    (at 26.055 56.78 270)
+    (at 25.2 55.9 180)
     (descr "Resistor SMD 0805 (2012 Metric), square (rectangular) end terminal, IPC_7351 nominal with elongated pad for handsoldering. (Body size source: https://docs.google.com/spreadsheets/d/1BsfQQcO9C6DZCsRaXUlFlo91Tg2WpOkGARC1WS5S8t0/edit?usp=sharing), generated with kicad-footprint-generator")
     (tags "resistor handsolder")
     (attr smd)
-    (fp_text reference R7 (at 0.02 -1.745 90) (layer F.SilkS)
-      (effects (font (size 1 1) (thickness 0.15)))
-    )
-    (fp_text value 10k (at 0 1.65 90) (layer F.Fab)
-      (effects (font (size 1 1) (thickness 0.15)))
-    )
-    (fp_text user %R (at 0 0 90) (layer F.Fab)
-      (effects (font (size 0.5 0.5) (thickness 0.08)))
-    )
-    (fp_line (start 1.85 0.95) (end -1.85 0.95) (layer F.CrtYd) (width 0.05))
-    (fp_line (start 1.85 -0.95) (end 1.85 0.95) (layer F.CrtYd) (width 0.05))
-    (fp_line (start -1.85 -0.95) (end 1.85 -0.95) (layer F.CrtYd) (width 0.05))
-    (fp_line (start -1.85 0.95) (end -1.85 -0.95) (layer F.CrtYd) (width 0.05))
-    (fp_line (start -0.261252 0.71) (end 0.261252 0.71) (layer F.SilkS) (width 0.12))
-    (fp_line (start -0.261252 -0.71) (end 0.261252 -0.71) (layer F.SilkS) (width 0.12))
-    (fp_line (start 1 0.6) (end -1 0.6) (layer F.Fab) (width 0.1))
-    (fp_line (start 1 -0.6) (end 1 0.6) (layer F.Fab) (width 0.1))
-    (fp_line (start -1 -0.6) (end 1 -0.6) (layer F.Fab) (width 0.1))
-    (fp_line (start -1 0.6) (end -1 -0.6) (layer F.Fab) (width 0.1))
-    (pad 2 smd roundrect (at 1.025 0 270) (size 1.15 1.4) (layers F.Cu F.Paste F.Mask) (roundrect_rratio 0.217391)
+    (fp_text reference R7 (at -2.7 0 90) (layer F.SilkS)
+      (effects (font (size 1 1) (thickness 0.15)))
+    )
+    (fp_text value 10k (at 0 1.65) (layer F.Fab)
+      (effects (font (size 1 1) (thickness 0.15)))
+    )
+    (fp_text user %R (at 0 0) (layer F.Fab)
+      (effects (font (size 0.5 0.5) (thickness 0.08)))
+    )
+    (fp_line (start 1.85 0.95) (end -1.85 0.95) (layer F.CrtYd) (width 0.05))
+    (fp_line (start 1.85 -0.95) (end 1.85 0.95) (layer F.CrtYd) (width 0.05))
+    (fp_line (start -1.85 -0.95) (end 1.85 -0.95) (layer F.CrtYd) (width 0.05))
+    (fp_line (start -1.85 0.95) (end -1.85 -0.95) (layer F.CrtYd) (width 0.05))
+    (fp_line (start -0.261252 0.71) (end 0.261252 0.71) (layer F.SilkS) (width 0.12))
+    (fp_line (start -0.261252 -0.71) (end 0.261252 -0.71) (layer F.SilkS) (width 0.12))
+    (fp_line (start 1 0.6) (end -1 0.6) (layer F.Fab) (width 0.1))
+    (fp_line (start 1 -0.6) (end 1 0.6) (layer F.Fab) (width 0.1))
+    (fp_line (start -1 -0.6) (end 1 -0.6) (layer F.Fab) (width 0.1))
+    (fp_line (start -1 0.6) (end -1 -0.6) (layer F.Fab) (width 0.1))
+    (pad 2 smd roundrect (at 1.025 0 180) (size 1.15 1.4) (layers F.Cu F.Paste F.Mask) (roundrect_rratio 0.217391)
       (net 15 +3V3))
-    (pad 1 smd roundrect (at -1.025 0 270) (size 1.15 1.4) (layers F.Cu F.Paste F.Mask) (roundrect_rratio 0.217391)
+    (pad 1 smd roundrect (at -1.025 0 180) (size 1.15 1.4) (layers F.Cu F.Paste F.Mask) (roundrect_rratio 0.217391)
       (net 45 RTC_IRQ))
     (model ${KISYS3DMOD}/Resistor_SMD.3dshapes/R_0805_2012Metric.wrl
@@
     (tags "resistor handsolder")
     (attr smd)
-    (fp_text reference R6 (at 0 -1.65 90) (layer F.SilkS)
+    (fp_text reference R6 (at 0.83 -1.65 90) (layer F.SilkS)
       (effects (font (size 1 1) (thickness 0.15)))
     )
@@
     (tags "resistor handsolder")
     (attr smd)
-    (fp_text reference R5 (at 0.2 1.8 90) (layer F.SilkS)
+    (fp_text reference R5 (at 0.855 1.8 90) (layer F.SilkS)
       (effects (font (size 1 1) (thickness 0.15)))
     )
@@
   (via (at 25.2 23.4) (size 0.8) (drill 0.4) (layers F.Cu B.Cu) (net 14))
   (via (at 46.2 51.8) (size 0.8) (drill 0.4) (layers F.Cu B.Cu) (net 14))
+  (via (at 44.9 33.2) (size 0.8) (drill 0.4) (layers F.Cu B.Cu) (net 14))
   (segment (start 38.3756 49.587) (end 38.8283 49.1343) (width 0.25) (layer F.Cu) (net 15))
   (segment (start 38.8283 49.1343) (end 40.1367 49.1343) (width 0.25) (layer F.Cu) (net 15))
@@
   (segment (start 29.58 51.4553) (end 28.4794 51.4553) (width 0.25) (layer F.Cu) (net 15))
   (segment (start 28.4794 51.4553) (end 28.03 51.9047) (width 0.25) (layer F.Cu) (net 15))
-  (segment (start 24.5927 52.73) (end 24.5927 56.3427) (width 0.25) (layer F.Cu) (net 15))
-  (segment (start 24.5927 56.3427) (end 26.055 57.805) (width 0.25) (layer F.Cu) (net 15))
   (segment (start 24.18 52.73) (end 24.5927 52.73) (width 0.25) (layer F.Cu) (net 15))
   (segment (start 29.58 50.58) (end 29.58 51.4553) (width 0.25) (layer F.Cu) (net 15))
@@
   (segment (start 44.37 53.13) (end 44.44 53.2) (width 0.25) (layer F.Cu) (net 15))
   (segment (start 44.44 53.2) (end 47.7 53.2) (width 0.25) (layer F.Cu) (net 15))
+  (segment (start 24.18 52.73) (end 24.18 55.88) (width 0.25) (layer F.Cu) (net 15))
   (segment (start 32.7122 44.4017) (end 32.4368 44.1263) (width 0.25) (layer F.Cu) (net 16))
   (segment (start 32.4368 44.1263) (end 32.3 44.1263) (width 0.25) (layer F.Cu) (net 16))
@@
   (segment (start 41.4534 44.4382) (end 37.2916 44.4382) (width 0.25) (layer B.Cu) (net 17))
   (via (at 37.2916 44.4382) (size 0.8) (layers F.Cu B.Cu) (net 17))
-  (segment (start 34.3 55.325) (end 38.8 59.825) (width 0.25) (layer F.Cu) (net 39))
-  (segment (start 38.8 59.825) (end 38.8 61.5) (width 0.25) (layer F.Cu) (net 39))
+  (segment (start 38.4 59.825) (end 38.4 61.5) (width 0.25) (layer F.Cu) (net 39))
+  (segment (start 34.3 55.325) (end 38.4 59.825) (width 0.25) (layer F.Cu) (net 39))
   (segment (start 39.455 50.1593) (end 40.0669 50.1593) (width 0.25) (layer F.Cu) (net 40))
   (segment (start 40.0669 50.1593) (end 43.1972 47.029) (width 0.25) (layer F.Cu) (net 40))

Commit message: update pcb
Routing:
- net GND: track 40.6 -> 36.9 mm
Changed lines of the file:
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@@
     (thickness 1.6)
     (drawings 23)
-    (tracks 319)
+    (tracks 318)
     (zones 0)
     (modules 42)
@@
   (segment (start 53.53 33.94) (end 53.53 32.7647) (width 0.25) (layer F.Cu) (net 14))
   (segment (start 27.33 52.78) (end 27.33 55.255) (width 0.25) (layer F.Cu) (net 14))
-  (segment (start 27.33 55.255) (end 29.9 57.825) (width 0.25) (layer F.Cu) (net 14))
   (segment (start 43.0723 71.0073) (end 43.16 71.095) (width 0.25) (layer F.Cu) (net 14))
   (segment (start 30.5 21.68) (end 30.5 22.2176) (width 0.25) (layer F.Cu) (net 14))
