File: HB-RF-MOD.kicad_pcb (KiCad board)
At the start: 2 copper layers, 35.6 x 64.2 mm, 42 parts, among them J1 RPi Header, J2 3V3, J3 GND, J4 RESET, J5 J_TCKC, J6 J_TMSC, Q1 BC847, Q2 BC847, Q3 BC847, Q4 BC847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

Commit message: update
Other:
- board text added: "A"
- board text added: "B"
- board text added: "G"
- board text added: "R"
Changed lines of the file:
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@@
   (general
     (thickness 1.6)
-    (drawings 23)
+    (drawings 27)
     (tracks 318)
     (zones 0)
@@
     (uvia_drill 0.1)
     (add_net +5V)
+  )
+  (module LED_THT:LED_D5.0mm-4_RGB_Wide_Pins (layer F.Cu)
+    (at 26.95 69.46 270)
+    (descr "LED, diameter 5.0mm, 2 pins, diameter 5.0mm, 3 pins, diameter 5.0mm, 4 pins, http://www.kingbright.com/attachments/file/psearch/000/00/00/L-154A4SUREQBFZGEW(Ver.9A).pdf")
+    (tags "LED diameter 5.0mm 2 pins diameter 5.0mm 3 pins diameter 5.0mm 4 pins RGB RGBLED")
+    (fp_text reference D1 (at 8.54 -0.25 270) (layer F.SilkS)
+      (effects (font (size 1 1) (thickness 0.15)))
+    )
+    (fp_text value LED_RGBA (at 3.2385 3.96 270) (layer F.Fab)
+      (effects (font (size 1 1) (thickness 0.15)))
+    )
+    (fp_text user %R (at 3.2385 -3.96 270) (layer F.Fab)
+      (effects (font (size 1 1) (thickness 0.15)))
+    )
+    (fp_line (start 7.56 -3.25) (end -1.08 -3.25) (layer F.CrtYd) (width 0.05))
+    (fp_line (start 7.56 3.25) (end 7.56 -3.25) (layer F.CrtYd) (width 0.05))
+    (fp_line (start -1.08 3.25) (end 7.56 3.25) (layer F.CrtYd) (width 0.05))
+    (fp_line (start -1.08 -3.25) (end -1.08 3.25) (layer F.CrtYd) (width 0.05))
+    (fp_line (start 0.6785 -1.545) (end 0.6785 -1.08) (layer F.SilkS) (width 0.12))
+    (fp_line (start 0.7385 -1.469694) (end 0.7385 1.469694) (layer F.Fab) (width 0.1))
+    (fp_circle (center 3.2385 0) (end 5.7385 0) (layer F.Fab) (width 0.1))
+    (fp_arc (start 3.2385 0) (end 0.983816 -1.08) (angle 128.8) (layer F.SilkS) (width 0.12))
+    (fp_arc (start 3.2385 0) (end 0.6785 -1.54483) (angle 127.7) (layer F.SilkS) (width 0.12))
+    (fp_arc (start 3.2385 0) (end 0.7385 -1.469694) (angle 299.1) (layer F.Fab) (width 0.1))
+    (pad 4 thru_hole circle (at 6.477 0 270) (size 1.8 1.8) (drill 0.9) (layers *.Cu *.Mask)
+      (net 42 +5V))
+    (pad 3 thru_hole circle (at 4.318 0 270) (size 1.8 1.8) (drill 0.9) (layers *.Cu *.Mask)
+      (net 50 "Net-(D1-Pad3)"))
+    (pad 2 thru_hole circle (at 2.159 0 270) (size 1.8 1.8) (drill 0.9) (layers *.Cu *.Mask)
+      (net 51 "Net-(D1-Pad2)"))
+    (pad 1 thru_hole rect (at 0 0 270) (size 1.8 1.8) (drill 0.9) (layers *.Cu *.Mask)
+      (net 52 "Net-(D1-Pad1)"))
+    (model ${KISYS3DMOD}/LED_THT.3dshapes/LED_D5.0mm-4_RGB_Wide_Pins.wrl
+      (at (xyz 0 0 0))
+      (scale (xyz 1 1 1))
+      (rotate (xyz 0 0 0))
+    )
   )
   (module additional:CP_Radial_D20.0mm_P5.00mm (layer B.Cu)
@@
     )
   )
-  (module LED_THT:LED_D5.0mm-4_RGB_Wide_Pins (layer F.Cu)
-    (at 26.95 69.46 270)
-    (descr "LED, diameter 5.0mm, 2 pins, diameter 5.0mm, 3 pins, diameter 5.0mm, 4 pins, http://www.kingbright.com/attachments/file/psearch/000/00/00/L-154A4SUREQBFZGEW(Ver.9A).pdf")
-    (tags "LED diameter 5.0mm 2 pins diameter 5.0mm 3 pins diameter 5.0mm 4 pins RGB RGBLED")
-    (fp_text reference D1 (at 8.54 -0.25 90) (layer F.SilkS)
-      (effects (font (size 1 1) (thickness 0.15)))
-    )
-    (fp_text value LED_RGBA (at 3.2385 3.96 90) (layer F.Fab)
-      (effects (font (size 1 1) (thickness 0.15)))
-    )
-    (fp_text user %R (at 3.2385 -3.96 90) (layer F.Fab)
-      (effects (font (size 1 1) (thickness 0.15)))
-    )
-    (fp_line (start 7.56 -3.25) (end -1.08 -3.25) (layer F.CrtYd) (width 0.05))
-    (fp_line (start 7.56 3.25) (end 7.56 -3.25) (layer F.CrtYd) (width 0.05))
-    (fp_line (start -1.08 3.25) (end 7.56 3.25) (layer F.CrtYd) (width 0.05))
-    (fp_line (start -1.08 -3.25) (end -1.08 3.25) (layer F.CrtYd) (width 0.05))
-    (fp_line (start 0.6785 1.08) (end 0.6785 1.545) (layer F.SilkS) (width 0.12))
-    (fp_line (start 0.6785 -1.545) (end 0.6785 -1.08) (layer F.SilkS) (width 0.12))
-    (fp_line (start 0.7385 -1.469694) (end 0.7385 1.469694) (layer F.Fab) (width 0.1))
-    (fp_circle (center 3.2385 0) (end 5.7385 0) (layer F.Fab) (width 0.1))
-    (fp_arc (start 3.2385 0) (end 0.983816 1.08) (angle -128.8) (layer F.SilkS) (width 0.12))
-    (fp_arc (start 3.2385 0) (end 0.983816 -1.08) (angle 128.8) (layer F.SilkS) (width 0.12))
-    (fp_arc (start 3.2385 0) (end 0.6785 1.54483) (angle -127.7) (layer F.SilkS) (width 0.12))
-    (fp_arc (start 3.2385 0) (end 0.6785 -1.54483) (angle 127.7) (layer F.SilkS) (width 0.12))
-    (fp_arc (start 3.2385 0) (end 0.7385 -1.469694) (angle 299.1) (layer F.Fab) (width 0.1))
-    (pad 4 thru_hole circle (at 6.477 0 270) (size 1.8 1.8) (drill 0.9) (layers *.Cu *.Mask)
-      (net 42 +5V))
-    (pad 3 thru_hole circle (at 4.318 0 270) (size 1.8 1.8) (drill 0.9) (layers *.Cu *.Mask)
-      (net 50 "Net-(D1-Pad3)"))
-    (pad 2 thru_hole circle (at 2.159 0 270) (size 1.8 1.8) (drill 0.9) (layers *.Cu *.Mask)
-      (net 51 "Net-(D1-Pad2)"))
-    (pad 1 thru_hole rect (at 0 0 270) (size 1.8 1.8) (drill 0.9) (layers *.Cu *.Mask)
-      (net 52 "Net-(D1-Pad1)"))
-    (model ${KISYS3DMOD}/LED_THT.3dshapes/LED_D5.0mm-4_RGB_Wide_Pins.wrl
-      (at (xyz 0 0 0))
-      (scale (xyz 1 1 1))
-      (rotate (xyz 0 0 0))
-    )
-  )
   (module additional:TRX2-TIF (layer F.Cu)
     (at 31.03 34.03 90)
@@
     )
   )
+  (gr_text A (at 24.7 75.95 90) (layer F.SilkS)
+    (effects (font (size 1.1 1.1) (thickness 0.2)))
+  )
+  (gr_text B (at 24.7 73.85 90) (layer F.SilkS)
+    (effects (font (size 1.1 1.1) (thickness 0.2)))
+  )
+  (gr_text G (at 24.7 71.65 90) (layer F.SilkS)
+    (effects (font (size 1.1 1.1) (thickness 0.2)))
+  )
+  (gr_text R (at 24.7 69.5 90) (layer F.SilkS)
+    (effects (font (size 1.1 1.1) (thickness 0.2)))
+  )
   (gr_line (start 45.1 23.7) (end 47.5 26.3) (layer F.SilkS) (width 0.15))
